File: PCB/JoyStick-Hat/JoyStick.kicad_sch (KiCad schematic)
At the start: 15 parts, among them J14 Conn_01x03_Pin, J15 Conn_01x03_Pin, J4 Conn_02x04_Odd_Even, J8 Conn_01x04_Pin, J9 Conn_01x04_Pin

Commit message: Board Routing
Connectors swapped around and board route started
Parts:
- removed J8, J9: Conn_01x04_Pin, Connector_PinHeader_2.54mm:PinHeader_1x04_P2.54mm_Vertical, symbol Connector:Conn_01x04_Pin
- added J8: Conn_02x04_Odd_Even, Connector_PinHeader_2.54mm:PinHeader_2x04_P2.54mm_Vertical, symbol Connector_Generic:Conn_02x04_Odd_Even
Connections:
- net GND: now also J8.2 (Pin_2), J8.7 (Pin_7)
- net ROTARY1_POLE1: now also J8.1 (Pin_1)
- net ROTARY1_POLE2: now also J8.3 (Pin_3)
- net ROTARY1_POLE3: now also J8.5 (Pin_5)
- net ROTARY2_POLE1: now also J8.8 (Pin_8)
- net ROTARY2_POLE2: now also J8.6 (Pin_6)
- net ROTARY2_POLE3: now also J8.4 (Pin_4)
Changed lines of the file:
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@@
   (junction (at 90.17 139.7) (diameter 0) (color 0 0 0 0)
   )
+  (wire (pts (xy 121.92 81.28) (xy 121.92 90.17))
+    (stroke (width 0) (type default))
+  )
   (wire (pts (xy 120.65 148.59) (xy 125.73 148.59))
     (stroke (width 0) (type default))
   )
-  (wire (pts (xy 63.5 95.25) (xy 109.22 95.25))
+  (wire (pts (xy 63.5 95.25) (xy 127 95.25))
     (stroke (width 0) (type default))
   )
@@
     (stroke (width 0) (type default))
   )
-  (wire (pts (xy 105.41 97.79) (xy 109.22 97.79))
+  (wire (pts (xy 105.41 97.79) (xy 129.54 97.79))
     (stroke (width 0) (type default))
   )
@@
     (stroke (width 0) (type default))
   )
-  (wire (pts (xy 57.15 92.71) (xy 109.22 92.71))
+  (wire (pts (xy 57.15 92.71) (xy 124.46 92.71))
     (stroke (width 0) (type default))
   )
@@
     (stroke (width 0) (type default))
   )
+  (wire (pts (xy 129.54 97.79) (xy 129.54 73.66))
+    (stroke (width 0) (type default))
+  )
+  (wire (pts (xy 124.46 92.71) (xy 124.46 78.74))
+    (stroke (width 0) (type default))
+  )
   (wire (pts (xy 120.65 114.3) (xy 120.65 148.59))
     (stroke (width 0) (type default))
@@
     (stroke (width 0) (type default))
   )
+  (wire (pts (xy 129.54 73.66) (xy 121.92 73.66))
+    (stroke (width 0) (type default))
+  )
+  (wire (pts (xy 127 95.25) (xy 127 76.2))
+    (stroke (width 0) (type default))
+  )
+  (wire (pts (xy 127 76.2) (xy 121.92 76.2))
+    (stroke (width 0) (type default))
+  )
   (wire (pts (xy 90.17 139.7) (xy 24.13 139.7))
     (stroke (width 0) (type default))
@@
     (stroke (width 0) (type default))
   )
-  (wire (pts (xy 50.8 90.17) (xy 109.22 90.17))
+  (wire (pts (xy 50.8 90.17) (xy 121.92 90.17))
     (stroke (width 0) (type default))
   )
   (wire (pts (xy 114.3 139.7) (xy 114.3 151.13))
+    (stroke (width 0) (type default))
+  )
+  (wire (pts (xy 124.46 78.74) (xy 121.92 78.74))
     (stroke (width 0) (type default))
   )
@@
     )
   )
-  (symbol (lib_id "Connector:Conn_01x04_Pin") (at 114.3 76.2 0) (mirror y) (unit 1)
-    (in_bom yes) (on_board yes) (dnp no)
-    (property "Reference" "J8" (at 114.3 71.12 0)
-      (effects (font (size 1.27 1.27)))
-    )
-    (property "Value" "Conn_01x04_Pin" (at 116.84 83.82 0)
-      (effects (font (size 1.27 1.27)))
-    )
-    (property "Footprint" "Connector_PinHeader_2.54mm:PinHeader_1x04_P2.54mm_Vertical" (at 114.3 76.2 0)
-      (effects (font (size 1.27 1.27)) hide)
-    )
-    (property "Datasheet" "~" (at 114.3 76.2 0)
-      (effects (font (size 1.27 1.27)) hide)
-    )
-    (pin "1")
-    (pin "2")
-    (pin "3")
-    (pin "4")
-    (instances
-      (project "JoyStick-Hat"
-        (path "/cf0c81b5-5bdf-47c3-83c0-f6980f515e65/657fac1d-f0e2-4536-8020-58a2ff4b82f6"
-          (reference "J8") (unit 1)
-        )
-      )
-    )
-  )
   (symbol (lib_id "power:+3.3V") (at 90.17 104.14 0) (mirror y) (unit 1)
     (in_bom yes) (on_board yes) (dnp no) (fields_autoplaced)
@@
     )
   )
-  (symbol (lib_id "Connector:Conn_01x04_Pin") (at 114.3 92.71 0) (mirror y) (unit 1)
-    (in_bom yes) (on_board yes) (dnp no)
-    (property "Reference" "J9" (at 114.3 87.63 0)
-      (effects (font (size 1.27 1.27)))
-    )
-    (property "Value" "Conn_01x04_Pin" (at 116.84 100.33 0)
-      (effects (font (size 1.27 1.27)))
-    )
-    (property "Footprint" "Connector_PinHeader_2.54mm:PinHeader_1x04_P2.54mm_Vertical" (at 114.3 92.71 0)
-      (effects (font (size 1.27 1.27)) hide)
-    )
-    (property "Datasheet" "~" (at 114.3 92.71 0)
-      (effects (font (size 1.27 1.27)) hide)
-    )
-    (pin "1")
-    (pin "2")
-    (pin "3")
-    (pin "4")
-    (instances
-      (project "JoyStick-Hat"
-        (path "/cf0c81b5-5bdf-47c3-83c0-f6980f515e65/657fac1d-f0e2-4536-8020-58a2ff4b82f6"
-          (reference "J9") (unit 1)
-        )
-      )
-    )
-  )
   (symbol (lib_id "power:GND") (at 105.41 81.28 0) (mirror y) (unit 1)
     (in_bom yes) (on_board yes) (dnp no) (fields_autoplaced)
@@
         )
       )
+    )
+  )
+  (symbol (lib_id "Connector_Generic:Conn_02x04_Odd_Even") (at 114.3 76.2 0) (unit 1)
+    (in_bom yes) (on_board yes) (dnp no) (fields_autoplaced)
+    (property "Reference" "J8" (at 115.57 67.31 0)
+      (effects (font (size 1.27 1.27)))
+    )
+    (property "Value" "Conn_02x04_Odd_Even" (at 115.57 69.85 0)
+      (effects (font (size 1.27 1.27)))
+    )
+    (property "Footprint" "Connector_PinHeader_2.54mm:PinHeader_2x04_P2.54mm_Vertical" (at 114.3 76.2 0)
+      (effects (font (size 1.27 1.27)) hide)
+    )
+    (property "Datasheet" "~" (at 114.3 76.2 0)
+      (effects (font (size 1.27 1.27)) hide)
+    )
+    (pin "4")
+    (pin "6")
+    (pin "7")
+    (pin "3")
+    (pin "5")
+    (pin "8")
+    (pin "2")
+    (pin "1")
+    (instances
+      (project "JoyStick-Hat"
+        (path "/cf0c81b5-5bdf-47c3-83c0-f6980f515e65/657fac1d-f0e2-4536-8020-58a2ff4b82f6"
+          (reference "J8") (unit 1)
+        )
+      )
