File: PCB/JoyStick-Hat/RPi_Interface.kicad_sch (KiCad schematic)
At the start: 19 parts, among them J7 Raspberry_Pi_2_3

Commit message: RJ45
Replaced RJ45 connector, original one had magnetics, those are not needed for RS485 and would have caused problems. Hooked up coms LEDs on RJ45 connector to MCU for debugging and displaying coms activity.
Parts:
- J7: footprint AVR-KiCAD-Lib-Connectors:PinHeader_2x21_P2.54mm_Female_Bottom -> AVR-KiCAD-Lib-Connectors:PinHeader_2x21_P2.54mm_Vertical
Changed lines of the file:
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@@
 			)
 		)
-		(property "Footprint" "AVR-KiCAD-Lib-Connectors:PinHeader_2x21_P2.54mm_Female_Bottom"
+		(property "Footprint" "AVR-KiCAD-Lib-Connectors:PinHeader_2x21_P2.54mm_Vertical"
 			(at 173.99 86.36 0)
 			(effects
