File: PCB/JoyStick-Hat/STM32F446RET6_MCU.kicad_sch (KiCad schematic)
At the start: 50 parts, among them J1 20021121-00010C4LF, J10 Conn_02x06_Odd_Even, J2 BU2032SM-JJ-GTR, J3 Conn_02x05_Odd_Even, SW1 TL3301NF260QG, U1 STM32F446VETx, X1 ABM3B-8.000MHZ-B2-T, X2 ABS07-32.768KHZ-9-T

Commit message: RJ45
Replaced RJ45 connector, original one had magnetics, those are not needed for RS485 and would have caused problems. Hooked up coms LEDs on RJ45 connector to MCU for debugging and displaying coms activity.
Connections:
- net RS485_RX_LED: now reaches U1.35 (PB0)
- net RS485_TX_LED: now reaches U1.36 (PB1)
Changed lines of the file:
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@@
+	(wire
+		(pts
+			(xy 161.29 91.44) (xy 137.16 91.44)
+		)
+		(stroke
+			(width 0)
+			(type default)
+		)
+	)
 	(wire
 		(pts
@@
 	(wire
 		(pts
+			(xy 266.7 78.74) (xy 158.75 78.74)
+		)
+		(stroke
+			(width 0)
+			(type default)
+		)
+	)
+	(wire
+		(pts
 			(xy 275.59 105.41) (xy 275.59 111.76)
 		)
@@
 	(wire
 		(pts
+			(xy 161.29 81.28) (xy 161.29 91.44)
+		)
+		(stroke
+			(width 0)
+			(type default)
+		)
+	)
+	(wire
+		(pts
 			(xy 175.26 29.21) (xy 182.88 29.21)
 		)
@@
 	(wire
 		(pts
+			(xy 158.75 78.74) (xy 158.75 88.9)
+		)
+		(stroke
+			(width 0)
+			(type default)
+		)
+	)
+	(wire
+		(pts
 			(xy 82.55 129.54) (xy 91.44 129.54)
 		)
@@
 	(wire
 		(pts
+			(xy 266.7 81.28) (xy 161.29 81.28)
+		)
+		(stroke
+			(width 0)
+			(type default)
+		)
+	)
+	(wire
+		(pts
 			(xy 271.78 86.36) (xy 275.59 86.36)
 		)
@@
 		(pts
 			(xy 16.51 121.92) (xy 22.86 121.92)
+		)
+		(stroke
+			(width 0)
+			(type default)
+		)
+	)
+	(wire
+		(pts
+			(xy 158.75 88.9) (xy 137.16 88.9)
 		)
 		(stroke
@@
 		)
 	)
+	(hierarchical_label "RS485_TX_LED"
+		(shape input)
+		(at 266.7 81.28 0)
+		(fields_autoplaced yes)
+		(effects
+			(font
+				(size 1.27 1.27)
+			)
+			(justify left)
+		)
+	)
 	(hierarchical_label "ROTARY1_POLE2"
 		(shape output)
@@
 		)
 	)
+	(hierarchical_label "RS485_RX_LED"
+		(shape input)
+		(at 266.7 78.74 0)
+		(fields_autoplaced yes)
+		(effects
+			(font
+				(size 1.27 1.27)
+			)
+			(justify left)
+		)
+	)
