File: PCB/JoyStick-Hat-V2-Re-Imagined/STM32F446RET6_MCU.kicad_sch (KiCad schematic)
At the start: 50 parts, among them J1 20021121-00010C4LF, J10 Conn_02x06_Odd_Even, J2 BU2032SM-JJ-GTR, J3 Conn_02x05_Odd_Even, SW1 TL3301NF260QG, U1 STM32F446VETx, X1 ABM3B-8.000MHZ-B2-T, X2 ABS07-32.768KHZ-9-T

Commit message: V2
Lots of progress made on version two of JoyStick Hat but the RPi 5 is going to be elimintated and an additional RS485 port added.
Parts:
- removed J10: Conn_02x06_Odd_Even, Connector_PinHeader_2.54mm:PinHeader_2x06_P2.54mm_Horizontal, symbol Connector_Generic:Conn_02x06_Odd_Even
- removed J3: Conn_02x05_Odd_Even, Connector_PinHeader_2.54mm:PinHeader_2x05_P2.54mm_Vertical, symbol Connector_Generic:Conn_02x05_Odd_Even
- removed SW1: TL3301NF260QG, AVR-KiCAD-Lib-Mech-Switches:TL3301NF260QG, symbol AVR-KiCAD-Lib-Mech-Switches:TL3301NF260QG
- added J3: 0901301210, AVR-KiCAD-Lib-Connectors:CON_901301210_MOL, symbol AVR-KiCAD-Lib-Connectors:0901301210
- added SW1: PTS636 SM43 SMTR LFS, AVR-KiCAD-Lib-Mech-Switches:PTS636 SM43 SMTR LFS, symbol AVR-KiCAD-Lib-Mech-Switches:PTS636 SM43 SMTR LFS
Connections:
- net +3.3V: now also J3.1, J3.2
- net GND: now also J3.10, J3.9, SW1.1
- net LED_DRIVER_BLANK: now also J3.8
- net LED_DRIVER_BLANK2: now also J3.6
- net LED_DRIVER_MOSI: now also J3.5
- net LED_DRIVER_SCLK: now also J3.3
- net LED_DRIVER_XLAT: now also J3.4
- net LED_DRIVER_XLAT2: now also J3.7
- net NRST: now also SW1.2
Other:
- note removed: "Diagnostic Serial Port - STM32"

Commit message: RPi Removed
Removed RPi from circuit added 20 pin JTAG schematic and PCB stil WIP
Parts:
- added J7: SBH11-PBPC-D10-ST-BK, AVR-KiCAD-Lib-Connectors:SULLINS_SBH11-PBPC-D10-ST-BK, symbol AVR-KiCAD-Lib-Connectors:SBH11-PBPC-D10-ST-BK
Connections:
- net +3.3V: now also J7.1
- net GND: now also J7.10, J7.12, J7.14, J7.16, J7.18, J7.2, J7.20, J7.4, J7.6, J7.8
- net NJTRST: now also J7.11
- net NRST: now also J7.13
- net SWCLK_TCK: now also J7.3
- net SWDIO_TMS: now also J7.5
- net SWO_TDI: now also J7.7
- net SWO_TDO: now also J7.9
- net at R14.1: no longer U1.93 (PB7)
- net at R15.1: no longer U1.95 (PB8)
- net at R16.1: no longer U1.96 (PB9)
- net at R12.1: no longer U1.91 (PB5)
- net at R13.1: no longer U1.92 (PB6)
- net ST_RPI_UART_CTS: no longer names the net of U1.70 (PA11)
- net ST_RPI_UART_RTS: no longer names the net of U1.71 (PA12)
- net ST_RPI_UART_RX: no longer names the net of U1.68 (PA9)
- net ST_RPI_UART_TX: no longer names the net of U1.69 (PA10)
- new net DBG_DBDI: J7.17, U1.92 (PB6)
- new net DBG_DBRQ: J7.15, U1.91 (PB5)
- no-connect marks 0 -> 1
