File: PCB/JoyStick-Hat-V2-Re-Imagined/STM32F446RET6_MCU.kicad_sch (KiCad schematic)
At the start: 61 parts, among them J1 20021121-00010C4LF, J10 0901301210, J12 DX07S016JA1R1500, J2 BU2032SM-JJ-GTR, J3 0901301210, J7 SBH11-PBPC-D10-ST-BK, SW1 PTS636 SM43 SMTR LFS, U1 STM32F446VETx, X1 ABM3B-8.000MHZ-B2-T, X2 ABS07-32.768KHZ-9-T

Commit message: Schematic Tweak
Making MCU page more readable
Parts:
- J10: footprint AVR-KiCAD-Lib-Connectors:CON_901301210_MOL -> AVR-KiCAD-Lib-Connectors:CON_901301212_MOL
Changed lines of the file:
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@@
 			)
 		)
-		(property "Footprint" "AVR-KiCAD-Lib-Connectors:CON_901301210_MOL"
+		(property "Footprint" "AVR-KiCAD-Lib-Connectors:CON_901301212_MOL"
 			(at 20.32 102.87 0)
 			(effects

Commit message: Schematic and board tweaks
tweaks to analog power section of MCU
Parts:
- added C22, C31: C0402C104K9PACTU, AVR-KiCAD-Lib-Resistors:R0402, symbol AVR-KiCAD-Lib-Capacitors:C0402C104K9PACTU
- added L5: BLM15HG601SN1D, AVR-KiCAD-Lib-Inductors:BLM15HG601SN1D, symbol AVR-KiCAD-Lib-Inductors:BLM15HG601SN1D
Connections:
- net +3.3V: now also C31.1, L5.1
- net GND: now also C22.2, C31.2
- net PE1: now reaches R9.1, U1.98 (PE1)
- net VCAP2: now reaches C23.1, C24.1, U1.73 (VCAP_2)
- net PA2: now reaches R19.1, U1.25 (PA2)
- net PE0: now reaches R8.1, U1.97 (PE0)
- net VREF+: now reaches U1.21 (VREF+)
- net VREF+: now also C22.1, L5.2
- net PD7: now reaches R10.1, U1.88 (PD7)
Other:
- moved on the sheet: C5, C6, J2, R1, R5, SW1
