File: PCB/LED_Driver_HUD/LED_Driver_HUD.kicad_pcb (KiCad board)
At the start: 4 copper layers, 60 x 85 mm, 15 parts, among them J1 Conn_02x05_Odd_Even, U1 TLC5947DAP, U2 TLC5947DAP

Commit message: LED HUD Complete
Added Additional indicator LEDs to LED HUD board. Full DRC pass.
Parts:
- added D10: HLMP-1401, AVR-KiCAD-Lib-Diodes:HLMP, F.Cu at (148.7, 63.0)
- added D11: HLMP-1401, AVR-KiCAD-Lib-Diodes:HLMP, F.Cu at (174.5, 71.8)
- added D12: HLMP-1401, AVR-KiCAD-Lib-Diodes:HLMP, F.Cu at (174.5, 76.0)
- added D5: HLMP-1401, AVR-KiCAD-Lib-Diodes:HLMP, F.Cu at (123.0, 71.8)
- added D6: HLMP-1401, AVR-KiCAD-Lib-Diodes:HLMP, F.Cu at (123.0, 76.1)
- added D7: HLMP-1401, AVR-KiCAD-Lib-Diodes:HLMP, F.Cu at (148.7, 67.4)
- added D8: HLMP-1401, AVR-KiCAD-Lib-Diodes:HLMP, F.Cu at (148.7, 71.8)
- added D9: HLMP-1401, AVR-KiCAD-Lib-Diodes:HLMP, F.Cu at (148.7, 58.6)
Connections:
- U1 pad 15: unconnected-(U1-OUT10-Pad15) -> Net-(U1-OUT10)
- U1 pad 16: unconnected-(U1-OUT11-Pad16) -> Net-(U1-OUT11)
- U1 pad 27: unconnected-(U1-OUT22-Pad27) -> Net-(U1-OUT22)
- U1 pad 28: unconnected-(U1-OUT23-Pad28) -> Net-(U1-OUT23)
- U2 pad 15: unconnected-(U2-OUT10-Pad15) -> Net-(U2-OUT10)
- U2 pad 16: unconnected-(U2-OUT11-Pad16) -> Net-(U2-OUT11)
- U2 pad 27: unconnected-(U2-OUT22-Pad27) -> Net-(U2-OUT22)
- U2 pad 28: unconnected-(U2-OUT23-Pad28) -> Net-(U2-OUT23)
Routing:
- net Net-(U2-OUT10): track 0.00 -> 70.3 mm
- net Net-(U2-OUT11): track 0.00 -> 66.6 mm
- net Net-(U1-OUT22): track 0.00 -> 61.4 mm, vias 0 -> 2
- net Net-(U2-OUT22): track 0.00 -> 57.3 mm, vias 0 -> 2
- net Net-(U1-OUT10): track 0.00 -> 57.0 mm
- net Net-(U1-OUT23): track 0.00 -> 54.7 mm, vias 0 -> 2
- net Net-(U1-OUT11): track 0.00 -> 53.3 mm
- net Net-(U2-OUT23): track 0.00 -> 50.4 mm, vias 0 -> 2
- net Net-(U2-OUT1): track 44.2 -> 43.2 mm
- net Net-(U2-OUT7): track 65.0 -> 64.0 mm
- net Net-(U2-OUT2): track 47.7 -> 46.7 mm
- net Net-(U2-OUT6): track 61.6 -> 60.6 mm
- net Net-(U2-OUT9): track 72.0 -> 71.0 mm
- net Net-(U2-OUT5): track 58.1 -> 57.1 mm
- net Net-(U2-OUT4): track 54.6 -> 53.6 mm
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
Commit message: Fab Fixes
Fixing for Frabrication, DRC cleared by pending external review subject to change.
Other:
- board text added: "3V3"
- board text added: "Accessibilita Project"
- board text added: "Designed by Adam Vadala-Roth"
- board text added: "GND"
- board text added: "GhostPCB LLC"
- board text added: "LED-Driver-HUD"
- board text added: "LED-Driver-HUD 0.1a 2024"
- board text added: "Mobility Independence Foundation"
- board text added: "PA4"
- board text added: "PA5"
- board text added: "PA6"
- board text added: "PA7"
- board text added: "PC4"
- board text added: "PC5"
- board text added: "https://github.com/Accessibilita"
